File: Hardware/ADS868_Test/ADS868_Test.kicad_pcb (KiCad board)
At the start: 2 copper layers, 50 x 44 mm, 27 parts, among them J101 Conn_01x01, J102 Conn_01x01, J103 Conn_01x01, J104 Conn_01x01, J105 71764-0012, J106 71764-0012, U101 ADS8681IPWR, U102 ADS8681IPWR, U103 LTC3525-5

Commit message: Design
Parts:
- moved J104 11.6 mm to (104.1, 88.9)
- moved J103 6.35 mm to (104.1, 78.7)
- moved J101 5.65 mm to (104.1, 58.4)
- moved J102 2.39 mm to (104.1, 68.6)
Changed lines of the file:
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@@
         (effects (font (size 1 1) (thickness 0.15)))
     )
-    (fp_text user "${REFERENCE}" (at 0 2.5 unlocked) (layer "F.Fab")
+    (fp_text user "${REFERENCE}" (at -0.031 2.364 unlocked) (layer "F.Fab")
         (effects (font (size 1 1) (thickness 0.15)))
     )
@@
   )
   (footprint "Connector_PinHeader_2.54mm:PinHeader_1x01_P2.54mm_Vertical" (layer "F.Cu")
-    (at 106.5 63.55)
+    (at 104.14 58.42)
     (descr "Through hole straight pin header, 1x01, 2.54mm pitch, single row")
     (tags "Through hole pin header THT 1x01 2.54mm single row")
@@
   )
   (footprint "Connector_PinHeader_2.54mm:PinHeader_1x01_P2.54mm_Vertical" (layer "F.Cu")
-    (at 106.5 77.5)
+    (at 104.14 88.9)
     (descr "Through hole straight pin header, 1x01, 2.54mm pitch, single row")
     (tags "Through hole pin header THT 1x01 2.54mm single row")
@@
   )
   (footprint "Connector_PinHeader_2.54mm:PinHeader_1x01_P2.54mm_Vertical" (layer "F.Cu")
-    (at 106.5 72.85)
+    (at 104.14 78.74)
     (descr "Through hole straight pin header, 1x01, 2.54mm pitch, single row")
     (tags "Through hole pin header THT 1x01 2.54mm single row")
@@
   )
   (footprint "Connector_PinHeader_2.54mm:PinHeader_1x01_P2.54mm_Vertical" (layer "F.Cu")
-    (at 106.5 68.2)
+    (at 104.14 68.58)
     (descr "Through hole straight pin header, 1x01, 2.54mm pitch, single row")
     (tags "Through hole pin header THT 1x01 2.54mm single row")

Commit message: Test
Parts:
- moved C109 94.4 mm to (136.5, 53.1), turned to 90 degrees
- moved R107 90.5 mm to (136.5, 56.5), turned to -90 degrees
- moved C105 84.6 mm to (123.6, 70.1)
- moved R103 84.0 mm to (127.1, 68.7), turned to 90 degrees
- moved C107 82.6 mm to (123.8, 87.0)
- moved R104 81.3 mm to (127.1, 85.7), turned to 90 degrees
- moved R106 79.6 mm to (127.1, 80.8), turned to -90 degrees
- moved R105 79.4 mm to (127.1, 63.9), turned to -90 degrees
- moved C110 78.7 mm to (129.3, 56.5), turned to -90 degrees
- moved R102 77.7 mm to (120.4, 87.0)
- moved C102 77.4 mm to (115.2, 85.1), turned to -90 degrees
- moved R101 76.6 mm to (120.1, 70.1)
- moved C103 76.2 mm to (114.9, 63.5), turned to -90 degrees
- moved C104 76.1 mm to (115.2, 80.5), turned to -90 degrees
- moved C101 75.7 mm to (114.9, 68.1), turned to -90 degrees
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Connections:
- J105 pad 10: unconnected-(J105-Pin_10-Pad10) -> /ADC1_SDI
- J105 pad 11: /ADC1_SDO-0 -> unconnected-(J105-Pin_11-Pad11)
- J105 pad 5: /ADC1_~{CS} -> /ADC1_RVS
- J105 pad 7: /ADC1_SCLK -> /ADC1_SDO-0
- J105 pad 8: /ADC1_RVS -> /ADC1_SCLK
- J105 pad 9: /ADC1_SDI -> /ADC1_~{CS}
- J106 pad 10: unconnected-(J106-Pin_10-Pad10) -> /ADC2_SDI
- J106 pad 11: /ADC2_SDO-0 -> unconnected-(J106-Pin_11-Pad11)
- J106 pad 5: /ADC2_~{CS} -> /ADC2_RVS
- J106 pad 7: /ADC2_SCLK -> /ADC2_SDO-0
- J106 pad 8: /ADC2_RVS -> /ADC2_SCLK
- J106 pad 9: /ADC2_SDI -> /ADC2_~{CS}
Routing:
- net +3V3: track 0.00 -> 89.7 mm, vias 0 -> 4
- net +5V: track 0.00 -> 43.8 mm, vias 0 -> 3
- net /ADC2_SDI: track 0.00 -> 21.9 mm
- net /ADC1_SDO-1: track 0.00 -> 21.3 mm
- net /ADC2_SCLK: track 0.00 -> 21.1 mm
- net /ADC2_SDO-1: track 0.00 -> 21.0 mm
- net /ADC1_SCLK: track 0.00 -> 20.8 mm
- net /ADC1_SDI: track 0.00 -> 20.8 mm
- net Net-(J101-Pin_1): track 0.00 -> 19.6 mm
- net /ADC1_RVS: track 0.00 -> 18.5 mm
- net /ADC2_~{CS}: track 0.00 -> 18.2 mm
- net /ADC2_SDO-0: track 0.00 -> 18.1 mm
- net /ADC1_SDO-0: track 0.00 -> 18.0 mm
- net /ADC1_~{CS}: track 0.00 -> 17.5 mm
- net /ADC2_RVS: track 0.00 -> 17.3 mm
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- added copper zone on B.Cu, net GND
- added copper zone on F.Cu, net GND
Other:
- board text added: "ADS8681_Test"
