File: Hardware/ADS868_Test/ADS868_Test.kicad_sch (KiCad schematic)
At the start: 27 parts, among them J1 71764-0012, J101 Conn_01x01, J102 Conn_01x01, J103 Conn_01x01, J104 Conn_01x01, J2 71764-0012, U103 LTC3525-5, U508 ADS8681IPWR

Commit message: Test
Connections:
- net ADC1_RVS: now also J1.5 (Pin_5); no longer J1.8 (Pin_8)
- net ADC1_SCLK: now also J1.8 (Pin_8); no longer J1.7 (Pin_7)
- net ADC1_SDI: now also J1.10 (Pin_10); no longer J1.9 (Pin_9)
- net ADC1_SDO-0: now also J1.7 (Pin_7); no longer J1.11 (Pin_11)
- net ADC1_~{CS}: now also J1.9 (Pin_9); no longer J1.5 (Pin_5)
- net ADC2_RVS: now also J2.5 (Pin_5); no longer J2.8 (Pin_8)
- net ADC2_SCLK: now also J2.8 (Pin_8); no longer J2.7 (Pin_7)
- net ADC2_SDI: now also J2.10 (Pin_10); no longer J2.9 (Pin_9)
- net ADC2_SDO-0: now also J2.7 (Pin_7); no longer J2.11 (Pin_11)
- net ADC2_~{CS}: now also J2.9 (Pin_9); no longer J2.5 (Pin_5)
Changed lines of the file:
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@@
   (junction (at 93.345 146.685) (diameter 0) (color 0 0 0 0)
   )
-  (no_connect (at 220.345 154.94))
+  (no_connect (at 207.645 157.48))
   (no_connect (at 267.335 157.48))
   (no_connect (at 220.345 157.48))
-  (no_connect (at 267.335 154.94))
+  (no_connect (at 254.635 157.48))
   (wire (pts (xy 70.485 130.175) (xy 56.515 130.175))
     (stroke (width 0) (type default))
@@
     (effects (font (size 1.27 1.27)) (justify left))
   )
-  (hierarchical_label "ADC1_~{CS}" (shape bidirectional) (at 207.645 149.86 180) (fields_autoplaced)
+  (hierarchical_label "ADC1_~{CS}" (shape bidirectional) (at 207.645 154.94 180) (fields_autoplaced)
     (effects (font (size 1.27 1.27)) (justify right))
   )
@@
     (effects (font (size 1.27 1.27)) (justify left))
   )
-  (hierarchical_label "ADC1_SDI" (shape bidirectional) (at 207.645 154.94 180) (fields_autoplaced)
-    (effects (font (size 1.27 1.27)) (justify right))
-  )
-  (hierarchical_label "ADC2_SCLK" (shape bidirectional) (at 254.635 152.4 180) (fields_autoplaced)
-    (effects (font (size 1.27 1.27)) (justify right))
+  (hierarchical_label "ADC1_SDI" (shape bidirectional) (at 220.345 154.94 0) (fields_autoplaced)
+    (effects (font (size 1.27 1.27)) (justify left))
+  )
+  (hierarchical_label "ADC2_SCLK" (shape bidirectional) (at 267.335 152.4 0) (fields_autoplaced)
+    (effects (font (size 1.27 1.27)) (justify left))
   )
   (hierarchical_label "ADC2_SDI" (shape bidirectional) (at 139.7 135.255 0) (fields_autoplaced)
@@
     (effects (font (size 1.27 1.27)) (justify left))
   )
-  (hierarchical_label "ADC2_SDO-0" (shape bidirectional) (at 254.635 157.48 180) (fields_autoplaced)
+  (hierarchical_label "ADC2_SDO-0" (shape bidirectional) (at 254.635 152.4 180) (fields_autoplaced)
     (effects (font (size 1.27 1.27)) (justify right))
   )
@@
     (effects (font (size 1.27 1.27)) (justify left))
   )
-  (hierarchical_label "ADC1_SDO-0" (shape bidirectional) (at 207.645 157.48 180) (fields_autoplaced)
+  (hierarchical_label "ADC1_SDO-0" (shape bidirectional) (at 207.645 152.4 180) (fields_autoplaced)
     (effects (font (size 1.27 1.27)) (justify right))
   )
@@
     (effects (font (size 1.27 1.27)) (justify left))
   )
-  (hierarchical_label "ADC1_SCLK" (shape bidirectional) (at 207.645 152.4 180) (fields_autoplaced)
-    (effects (font (size 1.27 1.27)) (justify right))
-  )
-  (hierarchical_label "ADC2_SDI" (shape bidirectional) (at 254.635 154.94 180) (fields_autoplaced)
-    (effects (font (size 1.27 1.27)) (justify right))
+  (hierarchical_label "ADC1_SCLK" (shape bidirectional) (at 220.345 152.4 0) (fields_autoplaced)
+    (effects (font (size 1.27 1.27)) (justify left))
+  )
+  (hierarchical_label "ADC2_SDI" (shape bidirectional) (at 267.335 154.94 0) (fields_autoplaced)
+    (effects (font (size 1.27 1.27)) (justify left))
   )
   (hierarchical_label "ADC1_SDO-1" (shape bidirectional) (at 135.89 74.93 0) (fields_autoplaced)
     (effects (font (size 1.27 1.27)) (justify left))
   )
-  (hierarchical_label "ADC2_RVS" (shape bidirectional) (at 267.335 152.4 0) (fields_autoplaced)
-    (effects (font (size 1.27 1.27)) (justify left))
-  )
-  (hierarchical_label "ADC2_~{CS}" (shape bidirectional) (at 254.635 149.86 180) (fields_autoplaced)
+  (hierarchical_label "ADC2_RVS" (shape bidirectional) (at 254.635 149.86 180) (fields_autoplaced)
+    (effects (font (size 1.27 1.27)) (justify right))
+  )
+  (hierarchical_label "ADC2_~{CS}" (shape bidirectional) (at 254.635 154.94 180) (fields_autoplaced)
     (effects (font (size 1.27 1.27)) (justify right))
   )
@@
     (effects (font (size 1.27 1.27)) (justify left))
   )
-  (hierarchical_label "ADC1_RVS" (shape bidirectional) (at 220.345 152.4 0) (fields_autoplaced)
-    (effects (font (size 1.27 1.27)) (justify left))
+  (hierarchical_label "ADC1_RVS" (shape bidirectional) (at 207.645 149.86 180) (fields_autoplaced)
+    (effects (font (size 1.27 1.27)) (justify right))
   )
   (symbol (lib_id "Connector_Generic:Conn_02x06_Odd_Even") (at 259.715 149.86 0) (unit 1)
@@
   (symbol (lib_id "Device:C") (at 106.045 111.76 90) (unit 1)
     (in_bom yes) (on_board yes) (dnp no)
-    (property "Reference" "C501" (at 107.315 105.41 90)
+    (property "Reference" "C501" (at 108.585 105.41 90)
       (effects (font (size 1.27 1.27)) (justify left))
     )
@@
     )
   )
-  (symbol (lib_id "power:+5V") (at 133.985 180.34 0) (unit 1)
-    (in_bom yes) (on_board yes) (dnp no)
-    (property "Reference" "#PWR0540" (at 133.985 184.15 0)
-      (effects (font (size 1.27 1.27)) hide)
-    )
-    (property "Value" "+5V" (at 134.366 175.9458 0)
-      (effects (font (size 1.27 1.27)))
-    )
-    (property "Footprint" "" (at 133.985 180.34 0)
-      (effects (font (size 1.27 1.27)) hide)
-    )
-    (property "Datasheet" "" (at 133.985 180.34 0)
-      (effects (font (size 1.27 1.27)) hide)
-    )
-    (pin "1")
-    (instances
-      (project "ETH3CDAQ1B.kicad_pcb"
-        (path "/9a321ea1-1f4e-4a89-b6fd-d20a870efce9/00000000-0000-0000-0000-00005fb85416"
-          (reference "#PWR0540") (unit 1)
-        )
-      )
-      (project "ADS868_Test"
-        (path "/cb9b19ae-2c54-4294-b7d8-04aca2d13600"
-          (reference "#PWR0119") (unit 1)
-        )
-      )
-    )
-  )
   (symbol (lib_id "power:+5V") (at 79.375 116.205 0) (unit 1)
     (in_bom yes) (on_board yes) (dnp no)
@@
         (path "/cb9b19ae-2c54-4294-b7d8-04aca2d13600"
           (reference "R107") (unit 1)
-        )
-      )
-    )
-  )
-  (symbol (lib_name "PWR_FLAG_1") (lib_id "power:PWR_FLAG") (at 133.985 180.34 180) (unit 1)
-    (in_bom yes) (on_board yes) (dnp no) (fields_autoplaced)
-    (property "Reference" "#FLG0103" (at 133.985 182.245 0)
-      (effects (font (size 1.27 1.27)) hide)
-    )
-    (property "Value" "PWR_FLAG" (at 133.985 184.785 0)
-      (effects (font (size 1.27 1.27)))
-    )
-    (property "Footprint" "" (at 133.985 180.34 0)
-      (effects (font (size 1.27 1.27)) hide)
-    )
-    (property "Datasheet" "~" (at 133.985 180.34 0)
-      (effects (font (size 1.27 1.27)) hide)
-    )
-    (pin "1")
-    (instances
-      (project "ADS868_Test"
-        (path "/cb9b19ae-2c54-4294-b7d8-04aca2d13600"
-          (reference "#FLG0103") (unit 1)
         )
       )
@@
   (symbol (lib_id "Device:C") (at 106.045 99.06 90) (unit 1)
     (in_bom yes) (on_board yes) (dnp no)
-    (property "Reference" "C502" (at 107.315 93.345 90)
-      (effects (font (size 1.27 1.27)) (justify left))
-    )
+    (property "Reference" "C502" (at 108.585 93.345 90)
+      (effects (font (size 1.27 1.27)) (justify left))
+    )
